File: PROJECTS/LAMP PROJECT/MICRO/MICRO_MODULAR_batt2.brd (EAGLE design)
At the start: 142.2 x 123.2 mm, 36 parts, among them J1 1X8, J2 1X8

Commit message: small modifications in some projects
Parts:
- moved J1 2.83 mm to (21.7, 80.2)
- moved J2 2.83 mm to (36.2, 80.2)
Routing:
- net SWITCH_BRAIN: track 117.5 -> 129.6 mm
